File: ControlBoard/ControlBoard.kicad_pcb (KiCad board)
At the start: 2 copper layers, 120 x 96.5 mm, 65 parts, among them IC1 PJA3404_R1_00001, IC2 PJA3404_R1_00001, IC3 PJA3404_R1_00001, IC4 PJA3404_R1_00001, J1 694106301002, Q1 NDS332P, Q10 NDS332P, Q12 NDS332P, Q2 NDS332P, Q3 NDS332P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

Commit message: Ordered
Parts:
- moved C3 45.7 mm to (161.4, 51.7), turned to 180 degrees
- moved C2 42.7 mm to (133.7, 88.0)
Connections:
- U2 pad 4: MUX0 -> unconnected-(U2-Pad4)
- U2 pad 5: MUX1 -> unconnected-(U2-Pad5)
- U2 pad 6: MUX2 -> unconnected-(U2-Pad6)
Routing:
- net GND: track 106.7 -> 97.9 mm
- net +5V: track 108.3 -> 102.9 mm
Other:
- board text added: "DC Train Control Board Designed by Michael Gamota 2022"
- board text removed: "DC Train Control Board Designed by Michael Gamota"
